Commit message: Modified the gripper's coordination as per the real robot

File: rain_description/urdf/rain_robot.urdf (robot description, URDF)
Before this commit: robot ur5_robotiq3, 52 links, 51 joints
Joints:
- joint r_robotiq_hand_joint: origin xyz=0.051 0 0 rpy=0 0 -1.57079632679 -> xyz=0.051 0 0 rpy=0 2.35619449019 -1.57079632679

Commit message: Added simulated webcams in gazebo

File: rain_description/urdf/rain_robot.urdf (robot description, URDF)
Before this commit: robot ur5_robotiq3, 52 links, 51 joints
Links:
- added link camera_link, mass 1e-5; collision box size=0.01 0.01 0.01; visual box size=0.01 0.01 0.01
- added link camera_link_front, mass 1e-5; collision box size=0.01 0.01 0.01; visual box size=0.01 0.01 0.01
- added link camera_link_top, mass 1e-5; collision box size=0.01 0.01 0.01; visual box size=0.01 0.01 0.01
Joints:
- removed joint fixed
- removed joint stand_joint
- added joint joint_stand_to_UR5: type fixed, parent stand, child base_link, origin xyz=0.0 0.0 1.0 rpy=0.0 0.0 0.0
- added joint joint_world_to_camera: type fixed, parent world, child camera_link, origin xyz=0.75 -1 1.2 rpy=0 0 1.57079632679, axis 0 1 0
- added joint joint_world_to_camera_front: type fixed, parent world, child camera_link_front, origin xyz=1.5 0 1.2 rpy=0 0 3.14159265359, axis 0 1 0
- added joint joint_world_to_camera_top: type fixed, parent world, child camera_link_top, origin xyz=0.75 0 2 rpy=0 1.57079632679 1.57079632679, axis 0 1 0
- added joint joint_world_to_stand: type fixed, parent world, child stand
