Commit message: Added a stand under the UR5 arm

File: rain_description/urdf/rain_robot.urdf.xacro (robot description, xacro)
@@ -2,4 +2,31 @@
 <robot xmlns:xacro="http://ros.org/wiki/xacro"
        name="ur5_robotiq3" >
+<!-- (0) Stand -->
+  <link name="world"/>
+  <!-- Stand -->
+  <link name="stand">
+    <inertial>
+        <mass value="1000" />
+        <origin xyz="0 0 0.5" rpy="0 0 0" />
+        <inertia ixx="0.01" ixy="0" ixz="0" iyy="0.01" iyz="0" izz="0.01" />
+    </inertial>
+    <visual>
+        <origin xyz="0 0 0.5" rpy="0 0 0" />
+        <geometry>
+            <cylinder length="1.0" radius="0.1" />
+        </geometry>
+    </visual>
+    <collision>
+        <origin xyz="0 0 0.5" rpy="0 0 0" />
+        <geometry>
+            <!-- <box size="0.2 0.2 1.0" /> -->
+            <cylinder length="1.0" radius="0.1" />
+        </geometry>
+    </collision>
+  </link>
+  <joint name="fixed" type="fixed">
+    <parent link="world"/>
+    <child link="stand"/>
+  </joint>
 <!-- (1) UR5 (extracted from "ur_description/ur5_upload.launch" from "universal_robot" package-->
   <!-- common stuff -->
@@ -9,9 +36,9 @@
   <!-- arm -->
   <xacro:ur5_robot prefix="" joint_limited="false"/>
-  <link name="world" />
-  <joint name="world_joint" type="fixed">
-    <parent link="world" />
+  <!-- <link name="world" /> -->
+  <joint name="stand_joint" type="fixed">
+    <parent link="stand" />
     <child link = "base_link" />
-    <origin xyz="0.0 0.0 0.0" rpy="0.0 0.0 0.0" />
+    <origin xyz="0.0 0.0 1.0" rpy="0.0 0.0 0.0" />
   </joint>
 <!-- (2) Robotiq 3-finger gripper (Right Hand) (added by Inmo) -->

Commit message: Modified to consider the real robot configuration

File: rain_description/urdf/rain_robot.urdf.xacro (robot description, xacro)
@@ -47,5 +47,5 @@
   <!-- gripper spawn: linking the gripper to the arm end effector -->
   <xacro:robotiq_hand prefix="r_" parent="ee_link" reflect="1">
-    <origin rpy="0 0 ${-pi/2.0}" xyz="0.051 0 0"/>
+    <origin rpy="0 ${pi/2.0 + pi/4.0} ${-pi/2.0}" xyz="0.051 0 0"/>
   </xacro:robotiq_hand>
   <gazebo>

Commit message: Simulated Camera Added in Gazebo

File: rain_description/urdf/rain_robot.urdf.xacro (robot description, xacro)
@@ -25,8 +25,216 @@
     </collision>
   </link>
-  <joint name="fixed" type="fixed">
+  <joint name="joint_world_to_stand" type="fixed">
     <parent link="world"/>
     <child link="stand"/>
   </joint>
+<!-- (0-A) Simulated Camera (Side View)-->
+  <xacro:property name="camera_size" value="0.01" />  <!-- Size of square 'camera' box -->
+  <!-- Camera -->
+  <link name="camera_link">
+    <collision>
+      <origin xyz="0 0 0" rpy="0 0 0"/>
+      <geometry>
+    <box size="${camera_size} ${camera_size} ${camera_size}"/>
+      </geometry>
+    </collision>
+    <visual>
+      <origin xyz="0 0 0" rpy="0 0 0"/>
+      <geometry>
+    <box size="${camera_size} ${camera_size} ${camera_size}"/>
+      </geometry>
+      <material name="red"/>
+    </visual>
+    <inertial>
+      <mass value="1e-5" />
+      <origin xyz="0 0 0" rpy="0 0 0"/>
+      <inertia ixx="1e-6" ixy="0" ixz="0" iyy="1e-6" iyz="0" izz="1e-6" />
+    </inertial>
+  </link>
+  <!-- camera position -->
+  <joint name="joint_world_to_camera" type="fixed">
+    <axis xyz="0 1 0" />
+    <origin xyz="0.75 -1 1.2" rpy="0 0 ${pi/2}"/>
+    <parent link="world"/>
+    <child link="camera_link"/>
+  </joint>
+  <!-- camera plugin -->
+  <gazebo reference="camera_link">
+    <sensor type="camera" name="camera1">
+      <update_rate>30.0</update_rate>
+      <camera name="head">
+        <horizontal_fov>1.3962634</horizontal_fov>
+        <image>
+          <width>800</width>
+          <height>800</height>
+          <format>R8G8B8</format>
+        </image>
+        <clip>
+          <near>0.02</near>
+          <far>300</far>
+        </clip>
+        <noise>
+          <type>gaussian</type>
+          <!-- Noise is sampled independently per pixel on each frame.
+               That pixel's noise value is added to each of its color
+               channels, which at that point lie in the range [0,1]. -->
+          <mean>0.0</mean>
+          <stddev>0.007</stddev>
+        </noise>
+      </camera>
+      <plugin name="camera_controller" filename="libgazebo_ros_camera.so">
+        <alwaysOn>true</alwaysOn>
+        <updateRate>0.0</updateRate>
+        <cameraName>camera1</cameraName>
+        <imageTopicName>image_raw</imageTopicName>
+        <cameraInfoTopicName>camera_info</cameraInfoTopicName>
+        <frameName>camera_link</frameName>
+        <hackBaseline>0.07</hackBaseline>
+        <distortionK1>0.0</distortionK1>
+        <distortionK2>0.0</distortionK2>
+        <distortionK3>0.0</distortionK3>
+        <distortionT1>0.0</distortionT1>
+        <distortionT2>0.0</distortionT2>
+      </plugin>
+    </sensor>
+  </gazebo>
+<!-- (0-B) Simulated Camera (Front View)-->
+  <!-- Camera -->
+  <link name="camera_link_front">
+    <collision>
+      <origin xyz="0 0 0" rpy="0 0 0"/>
+      <geometry>
+    <box size="${camera_size} ${camera_size} ${camera_size}"/>
+      </geometry>
+    </collision>
+    <visual>
+      <origin xyz="0 0 0" rpy="0 0 0"/>
+      <geometry>
+    <box size="${camera_size} ${camera_size} ${camera_size}"/>
+      </geometry>
+      <material name="red"/>
+    </visual>
+    <inertial>
+      <mass value="1e-5" />
+      <origin xyz="0 0 0" rpy="0 0 0"/>
+      <inertia ixx="1e-6" ixy="0" ixz="0" iyy="1e-6" iyz="0" izz="1e-6" />
+    </inertial>
+  </link>
+  <!-- camera position -->
+  <joint name="joint_world_to_camera_front" type="fixed">
+    <axis xyz="0 1 0" />
+    <origin xyz="1.5 0 1.2" rpy="0 0 ${pi}"/>
+    <parent link="world"/>
+    <child link="camera_link_front"/>
+  </joint>
+  <!-- camera plugin -->
+  <gazebo reference="camera_link_front">
+    <sensor type="camera" name="camera2">
+      <update_rate>30.0</update_rate>
+      <camera name="head">
+        <horizontal_fov>1.3962634</horizontal_fov>
+        <image>
+          <width>800</width>
+          <height>800</height>
+          <format>R8G8B8</format>
+        </image>
+        <clip>
+          <near>0.02</near>
+          <far>300</far>
+        </clip>
+        <noise>
+          <type>gaussian</type>
+          <!-- Noise is sampled independently per pixel on each frame.
+               That pixel's noise value is added to each of its color
+               channels, which at that point lie in the range [0,1]. -->
+          <mean>0.0</mean>
+          <stddev>0.007</stddev>
+        </noise>
+      </camera>
+      <plugin name="camera_controller" filename="libgazebo_ros_camera.so">
+        <alwaysOn>true</alwaysOn>
+        <updateRate>0.0</updateRate>
+        <cameraName>camera2</cameraName>
+        <imageTopicName>image_raw</imageTopicName>
+        <cameraInfoTopicName>front_camera_info</cameraInfoTopicName>
+        <frameName>front_camera_link</frameName>
+        <hackBaseline>0.07</hackBaseline>
+        <distortionK1>0.0</distortionK1>
+        <distortionK2>0.0</distortionK2>
+        <distortionK3>0.0</distortionK3>
+        <distortionT1>0.0</distortionT1>
+        <distortionT2>0.0</distortionT2>
+      </plugin>
+    </sensor>
+  </gazebo>
+<!-- (0-C) Simulated Camera (Top View)-->
+  <!-- Camera -->
+  <link name="camera_link_top">
+    <collision>
+      <origin xyz="0 0 0" rpy="0 0 0"/>
+      <geometry>
+    <box size="${camera_size} ${camera_size} ${camera_size}"/>
+      </geometry>
+    </collision>
+    <visual>
+      <origin xyz="0 0 0" rpy="0 0 0"/>
+      <geometry>
+    <box size="${camera_size} ${camera_size} ${camera_size}"/>
+      </geometry>
+      <material name="red"/>
+    </visual>
+    <inertial>
+      <mass value="1e-5" />
+      <origin xyz="0 0 0" rpy="0 0 0"/>
+      <inertia ixx="1e-6" ixy="0" ixz="0" iyy="1e-6" iyz="0" izz="1e-6" />
+    </inertial>
+  </link>
+  <!-- camera position -->
+  <joint name="joint_world_to_camera_top" type="fixed">
+    <axis xyz="0 1 0" />
+    <origin xyz="0.75 0 2" rpy="0 ${pi/2} ${pi/2}"/>
+    <parent link="world"/>
+    <child link="camera_link_top"/>
+  </joint>
+  <!-- camera plugin -->
+  <gazebo reference="camera_link_top">
+    <sensor type="camera" name="camera3">
+      <update_rate>30.0</update_rate>
+      <camera name="head">
+        <horizontal_fov>1.3962634</horizontal_fov>
+        <image>
+          <width>800</width>
+          <height>800</height>
+          <format>R8G8B8</format>
+        </image>
+        <clip>
+          <near>0.02</near>
+          <far>300</far>
+        </clip>
+        <noise>
+          <type>gaussian</type>
+          <!-- Noise is sampled independently per pixel on each frame.
+               That pixel's noise value is added to each of its color
+               channels, which at that point lie in the range [0,1]. -->
+          <mean>0.0</mean>
+          <stddev>0.007</stddev>
+        </noise>
+      </camera>
+      <plugin name="camera_controller" filename="libgazebo_ros_camera.so">
+        <alwaysOn>true</alwaysOn>
+        <updateRate>0.0</updateRate>
+        <cameraName>camera3</cameraName>
+        <imageTopicName>image_raw</imageTopicName>
+        <cameraInfoTopicName>top_camera_info</cameraInfoTopicName>
+        <frameName>top_camera_link</frameName>
+        <hackBaseline>0.07</hackBaseline>
+        <distortionK1>0.0</distortionK1>
+        <distortionK2>0.0</distortionK2>
+        <distortionK3>0.0</distortionK3>
+        <distortionT1>0.0</distortionT1>
+        <distortionT2>0.0</distortionT2>
+      </plugin>
+    </sensor>
+  </gazebo>
 <!-- (1) UR5 (extracted from "ur_description/ur5_upload.launch" from "universal_robot" package-->
   <!-- common stuff -->
@@ -37,5 +245,5 @@
   <xacro:ur5_robot prefix="" joint_limited="false"/>
   <!-- <link name="world" /> -->
-  <joint name="stand_joint" type="fixed">
+  <joint name="joint_stand_to_UR5" type="fixed">
     <parent link="stand" />
     <child link = "base_link" />

Commit message: Refactoring

File: rain_description/urdf/rain_robot.urdf.xacro (robot description, xacro)
@@ -29,234 +29,26 @@
     <child link="stand"/>
   </joint>
-<!-- (0-A) Simulated Camera (Side View)-->
-  <xacro:property name="camera_size" value="0.01" />  <!-- Size of square 'camera' box -->
-  <!-- Camera -->
-  <link name="camera_link">
-    <collision>
-      <origin xyz="0 0 0" rpy="0 0 0"/>
-      <geometry>
-    <box size="${camera_size} ${camera_size} ${camera_size}"/>
-      </geometry>
-    </collision>
-    <visual>
-      <origin xyz="0 0 0" rpy="0 0 0"/>
-      <geometry>
-    <box size="${camera_size} ${camera_size} ${camera_size}"/>
-      </geometry>
-      <material name="red"/>
-    </visual>
-    <inertial>
-      <mass value="1e-5" />
-      <origin xyz="0 0 0" rpy="0 0 0"/>
-      <inertia ixx="1e-6" ixy="0" ixz="0" iyy="1e-6" iyz="0" izz="1e-6" />
-    </inertial>
-  </link>
-  <!-- camera position -->
-  <joint name="joint_world_to_camera" type="fixed">
-    <axis xyz="0 1 0" />
-    <origin xyz="0.75 -1 1.2" rpy="0 0 ${pi/2}"/>
-    <parent link="world"/>
-    <child link="camera_link"/>
-  </joint>
-  <!-- camera plugin -->
-  <gazebo reference="camera_link">
-    <sensor type="camera" name="usb_cam_1">
-      <update_rate>30.0</update_rate>
-      <camera name="head">
-        <horizontal_fov>1.3962634</horizontal_fov>
-        <image>
-          <width>800</width>
-          <height>800</height>
-          <format>R8G8B8</format>
-        </image>
-        <clip>
-          <near>0.02</near>
-          <far>300</far>
-        </clip>
-        <noise>
-          <type>gaussian</type>
-          <!-- Noise is sampled independently per pixel on each frame.
-               That pixel's noise value is added to each of its color
-               channels, which at that point lie in the range [0,1]. -->
-          <mean>0.0</mean>
-          <stddev>0.007</stddev>
-        </noise>
-      </camera>
-      <plugin name="camera_controller" filename="libgazebo_ros_camera.so">
-        <alwaysOn>true</alwaysOn>
-        <updateRate>0.0</updateRate>
-        <cameraName>usb_cam_1</cameraName>
-        <imageTopicName>image_raw</imageTopicName>
-        <cameraInfoTopicName>camera_info</cameraInfoTopicName>
-        <frameName>camera_link</frameName>
-        <hackBaseline>0.07</hackBaseline>
-        <distortionK1>0.0</distortionK1>
-        <distortionK2>0.0</distortionK2>
-        <distortionK3>0.0</distortionK3>
-        <distortionT1>0.0</distortionT1>
-        <distortionT2>0.0</distortionT2>
-      </plugin>
-    </sensor>
-  </gazebo>
-<!-- (0-B) Simulated Camera (Front View)-->
-  <!-- Camera -->
-  <link name="camera_link_front">
-    <collision>
-      <origin xyz="0 0 0" rpy="0 0 0"/>
-      <geometry>
-    <box size="${camera_size} ${camera_size} ${camera_size}"/>
-      </geometry>
-    </collision>
-    <visual>
-      <origin xyz="0 0 0" rpy="0 0 0"/>
-      <geometry>
-    <box size="${camera_size} ${camera_size} ${camera_size}"/>
-      </geometry>
-      <material name="red"/>
-    </visual>
-    <inertial>
-      <mass value="1e-5" />
-      <origin xyz="0 0 0" rpy="0 0 0"/>
-      <inertia ixx="1e-6" ixy="0" ixz="0" iyy="1e-6" iyz="0" izz="1e-6" />
-    </inertial>
-  </link>
-  <!-- camera position -->
-  <joint name="joint_world_to_camera_front" type="fixed">
-    <axis xyz="0 1 0" />
-    <origin xyz="1.5 0 1.2" rpy="0 0 ${pi}"/>
-    <parent link="world"/>
-    <child link="camera_link_front"/>
-  </joint>
-  <!-- camera plugin -->
-  <gazebo reference="camera_link_front">
-    <sensor type="camera" name="usb_cam_2">
-      <update_rate>30.0</update_rate>
-      <camera name="head">
-        <horizontal_fov>1.3962634</horizontal_fov>
-        <image>
-          <width>800</width>
-          <height>800</height>
-          <format>R8G8B8</format>
-        </image>
-        <clip>
-          <near>0.02</near>
-          <far>300</far>
-        </clip>
-        <noise>
-          <type>gaussian</type>
-          <!-- Noise is sampled independently per pixel on each frame.
-               That pixel's noise value is added to each of its color
-               channels, which at that point lie in the range [0,1]. -->
-          <mean>0.0</mean>
-          <stddev>0.007</stddev>
-        </noise>
-      </camera>
-      <plugin name="camera_controller" filename="libgazebo_ros_camera.so">
-        <alwaysOn>true</alwaysOn>
-        <updateRate>0.0</updateRate>
-        <cameraName>usb_cam_2</cameraName>
-        <imageTopicName>image_raw</imageTopicName>
-        <cameraInfoTopicName>front_camera_info</cameraInfoTopicName>
-        <frameName>front_camera_link</frameName>
-        <hackBaseline>0.07</hackBaseline>
-        <distortionK1>0.0</distortionK1>
-        <distortionK2>0.0</distortionK2>
-        <distortionK3>0.0</distortionK3>
-        <distortionT1>0.0</distortionT1>
-        <distortionT2>0.0</distortionT2>
-      </plugin>
-    </sensor>
-  </gazebo>
-<!-- (0-C) Simulated Camera (Top View)-->
-  <!-- Camera -->
-  <link name="camera_link_top">
-    <collision>
-      <origin xyz="0 0 0" rpy="0 0 0"/>
-      <geometry>
-    <box size="${camera_size} ${camera_size} ${camera_size}"/>
-      </geometry>
-    </collision>
-    <visual>
-      <origin xyz="0 0 0" rpy="0 0 0"/>
-      <geometry>
-    <box size="${camera_size} ${camera_size} ${camera_size}"/>
-      </geometry>
-      <material name="red"/>
-    </visual>
-    <inertial>
-      <mass value="1e-5" />
-      <origin xyz="0 0 0" rpy="0 0 0"/>
-      <inertia ixx="1e-6" ixy="0" ixz="0" iyy="1e-6" iyz="0" izz="1e-6" />
-    </inertial>
-  </link>
-  <!-- camera position -->
-  <joint name="joint_world_to_camera_top" type="fixed">
-    <axis xyz="0 1 0" />
-    <origin xyz="0.75 0 2" rpy="0 ${pi/2} ${pi/2}"/>
-    <parent link="world"/>
-    <child link="camera_link_top"/>
-  </joint>
-  <!-- camera plugin -->
-  <gazebo reference="camera_link_top">
-    <sensor type="camera" name="usb_cam_3">
-      <update_rate>30.0</update_rate>
-      <camera name="head">
-        <horizontal_fov>1.3962634</horizontal_fov>
-        <image>
-          <width>800</width>
-          <height>800</height>
-          <format>R8G8B8</format>
-        </image>
-        <clip>
-          <near>0.02</near>
-          <far>300</far>
-        </clip>
-        <noise>
-          <type>gaussian</type>
-          <!-- Noise is sampled independently per pixel on each frame.
-               That pixel's noise value is added to each of its color
-               channels, which at that point lie in the range [0,1]. -->
-          <mean>0.0</mean>
-          <stddev>0.007</stddev>
-        </noise>
-      </camera>
-      <plugin name="camera_controller" filename="libgazebo_ros_camera.so">
-        <alwaysOn>true</alwaysOn>
-        <updateRate>0.0</updateRate>
-        <cameraName>usb_cam_3</cameraName>
-        <imageTopicName>image_raw</imageTopicName>
-        <cameraInfoTopicName>top_camera_info</cameraInfoTopicName>
-        <frameName>top_camera_link</frameName>
-        <hackBaseline>0.07</hackBaseline>
-        <distortionK1>0.0</distortionK1>
-        <distortionK2>0.0</distortionK2>
-        <distortionK3>0.0</distortionK3>
-        <distortionT1>0.0</distortionT1>
-        <distortionT2>0.0</distortionT2>
-      </plugin>
-    </sensor>
-  </gazebo>
 <!-- (1) UR5 (extracted from "ur_description/ur5_upload.launch" from "universal_robot" package-->
   <!-- common stuff -->
-  <xacro:include filename="$(find ur_description)/urdf/common.gazebo.xacro" />
+  <xacro:include filename="$(find rain_description)/urdf/common.gazebo.xacro" />
+  <!-- (A) Bring a Robotic System -->
   <!-- ur5 -->
   <xacro:include filename="$(find ur_description)/urdf/ur5.urdf.xacro" />
-  <!-- arm -->
+  <!-- 3 finger robotiq gripper -->
+  <!-- <xacro:include filename="$(find robotiq_description)/urdf/robotiq_hand.urdf.xacro" /> -->
+  <!-- (B) Spawn the robot model (Right Arm) -->
+  <!-- ur5 -->
   <xacro:ur5_robot prefix="" joint_limited="false"/>
-  <!-- <link name="world" /> -->
   <joint name="joint_stand_to_UR5" type="fixed">
     <parent link="stand" />
     <child link = "base_link" />
-    <origin xyz="0.0 0.0 1.0" rpy="0.0 0.0 0.0" />
+    <origin xyz="0.0 0.0 1.01" rpy="0.0 0.0 0.0" />
   </joint>
-<!-- (2) Robotiq 3-finger gripper (Right Hand) (added by Inmo) -->
-  <!-- gripper -->
-  <xacro:include filename="$(find robotiq_description)/urdf/robotiq_hand.urdf.xacro" />
   <!-- gripper spawn: linking the gripper to the arm end effector -->
-  <xacro:robotiq_hand prefix="r_" parent="ee_link" reflect="1">
+  <!-- <xacro:robotiq_hand prefix="" parent="ee_link" reflect="1">
     <origin rpy="0 ${pi/2.0 + pi/4.0} ${-pi/2.0}" xyz="0.051 0 0"/>
-  </xacro:robotiq_hand>
-  <gazebo>
-    <!-- plugin for left RobotiQ hand -->
+  </xacro:robotiq_hand> -->
+  <!-- plugin for RobotiQ hands -->
+  <!-- <gazebo>
     <plugin name="left_robotiq_hand_plugin" filename="libRobotiqHandPlugin.so">
       <side>left</side>
@@ -264,5 +56,4 @@
       <kd_position>0.5</kd_position>
     </plugin>
-    <!-- plugin for right RobotiQ hand -->
     <plugin name="right_robotiq_hand_plugin" filename="libRobotiqHandPlugin.so">
       <side>right</side>
@@ -270,4 +61,4 @@
       <kd_position>0.5</kd_position>
     </plugin>
-  </gazebo>
+  </gazebo> -->
 </robot>
