Commit message: Refactored launch files

File: rain_description/urdf/rain_test_env.urdf.xacro (robot description, xacro)
@@ -1,4 +1,4 @@
 <?xml version="1.0"?>
-<test_env xmlns:xacro="http://ros.org/wiki/xacro"
+<robot xmlns:xacro="http://ros.org/wiki/xacro"
        name="rain_test_env" >
 <!-- (0) Stand -->
@@ -212,3 +212,3 @@
     </sensor>
   </gazebo>
-</test_env>
+</robot>

File: rain_description/urdf/rain_ur5_limited.urdf.xacro (robot description, xacro)
@@ -49,24 +49,3 @@
     <origin xyz="0.0 0.0 1.0" rpy="0.0 0.0 0.0" />
   </joint>
-<!-- (2) Robotiq 3-finger gripper (Right Hand) (added by Inmo) -->
-  <!-- gripper -->
-  <xacro:include filename="$(find robotiq_description)/urdf/robotiq_hand.urdf.xacro" />
-  <!-- gripper spawn: linking the gripper to the arm end effector -->
-  <xacro:robotiq_hand prefix="r_" parent="ee_link" reflect="1">
-    <origin rpy="0 0 ${-pi/2.0}" xyz="0.051 0 0"/>
-  </xacro:robotiq_hand>
-  <gazebo>
-    <!-- plugin for left RobotiQ hand -->
-    <plugin name="left_robotiq_hand_plugin" filename="libRobotiqHandPlugin.so">
-      <side>left</side>
-      <kp_position>10.0</kp_position>
-      <kd_position>0.5</kd_position>
-    </plugin>
-    <!-- plugin for right RobotiQ hand -->
-    <plugin name="right_robotiq_hand_plugin" filename="libRobotiqHandPlugin.so">
-      <side>right</side>
-      <kp_position>10.0</kp_position>
-      <kd_position>0.5</kd_position>
-    </plugin>
-  </gazebo>
 </robot>

File: rain_description/urdf/rain_ur5_robotiq3f.urdf.xacro (robot description, xacro)
@@ -36,5 +36,5 @@
   <xacro:include filename="$(find ur_description)/urdf/ur5.urdf.xacro" />
   <!-- 3 finger robotiq gripper -->
-  <!-- <xacro:include filename="$(find robotiq_description)/urdf/robotiq_hand.urdf.xacro" /> -->
+  <xacro:include filename="$(find robotiq_description)/urdf/robotiq_hand.urdf.xacro" />
   <!-- (B) Spawn the robot model (Right Arm) -->
   <!-- ur5 -->
@@ -46,9 +46,9 @@
   </joint>
   <!-- gripper spawn: linking the gripper to the arm end effector -->
-  <!-- <xacro:robotiq_hand prefix="" parent="ee_link" reflect="1">
+  <xacro:robotiq_hand prefix="" parent="ee_link" reflect="1">
     <origin rpy="0 ${pi/2.0 + pi/4.0} ${-pi/2.0}" xyz="0.051 0 0"/>
-  </xacro:robotiq_hand> -->
+  </xacro:robotiq_hand>
   <!-- plugin for RobotiQ hands -->
-  <!-- <gazebo>
+  <gazebo>
     <plugin name="left_robotiq_hand_plugin" filename="libRobotiqHandPlugin.so">
       <side>left</side>
@@ -61,4 +61,4 @@
       <kd_position>0.5</kd_position>
     </plugin>
-  </gazebo> -->
+  </gazebo>
 </robot>
